Commit message: Update URDF

File: robot.xacro (robot description, xacro)
@@ -25,10 +25,10 @@
     <parent link="base_link"/>
     <child link="imu_link"/>
-    <origin xyz="-0.0582085 -0.079396 0.228256" rpy="${pi/2} ${pi/2} 0.0"/>
+    <origin xyz="-0.04281711 -0.12469021 0.21492789" rpy="${pi/2} ${-pi/2} 0.0"/>
   </joint>
   <joint name="base_camera" type="fixed">
     <parent link="base_link"/>
     <child link="camera_link"/>
-    <origin xyz="0.117094 0.0 0.087219"/>
+    <origin xyz="0.11784511 0.0 0.09754467"/>
   </joint>
   <joint name="camera_optical_joint" type="fixed">

Commit message: AprilTag launch file

File: robot.xacro (robot description, xacro)
@@ -21,5 +21,5 @@
   <link name="imu_link"/>
   <link name="camera_link"/>
-  <link name="camera_link_optical"/>
+  <link name="camera"/>
   <joint name="base_imu" type="fixed">
     <parent link="base_link"/>
@@ -34,5 +34,5 @@
   <joint name="camera_optical_joint" type="fixed">
       <parent link="camera_link"/>
-      <child link="camera_link_optical"/>
+      <child link="camera"/>
       <origin xyz="0 0 0" rpy="${-pi/2} 0 ${-pi/2}"/>
     </joint>

Commit message: update URDF

File: robot.xacro (robot description, xacro)
@@ -13,5 +13,5 @@
       <origin xyz="${length/2 -0.01525722} ${width/2 -0.05384791} 0.0" rpy="0 0 ${-pi/2}" />
       <geometry>
-        <mesh filename="file://ROOT.stl"/>
+        <mesh filename="ROOT.stl"/>
         <box size="0.23495 0.269875 0.293653"/>
       </geometry>

Commit message: Try pose estimation

File: robot.xacro (robot description, xacro)
@@ -30,5 +30,5 @@
     <parent link="base_link"/>
     <child link="camera_link"/>
-    <origin xyz="0.11784511 0.0 0.09754467"/>
+    <origin xyz="0.11784511 0.0 0.09754467" rpy="${pi} 0 0"/>
   </joint>
   <joint name="camera_optical_joint" type="fixed">
